File: week 1/Motor Slave_+_IMU sensor/Motor Slave_+_IMU sensor.sch (EAGLE design)
At the start: 8 parts

Commit message: .
Connections:
- net PA_11: no longer ENCODER.1
- net PA_12: no longer ENCODER.2
- net PB_3: now also ENCODER.1
- net PB_4: now also ENCODER.2
Changed lines of the file:
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@@
 <label x="33.02" y="71.12" size="1.778" layer="95" rot="R180" xref="yes"/>
-</segment>
-<segment>
-<pinref part="ENCODER" gate="A" pin="1"/>
-<wire x1="7.62" y1="55.88" x2="12.7" y2="55.88" width="0.1524" layer="91"/>
-<label x="12.7" y="55.88" size="1.778" layer="95" xref="yes"/>
 </segment>
 </net>
@@
 <wire x1="38.1" y1="66.04" x2="33.02" y2="66.04" width="0.1524" layer="91"/>
 <label x="33.02" y="66.04" size="1.778" layer="95" rot="R180" xref="yes"/>
-</segment>
-<segment>
-<pinref part="ENCODER" gate="A" pin="2"/>
-<wire x1="7.62" y1="58.42" x2="12.7" y2="58.42" width="0.1524" layer="91"/>
-<label x="12.7" y="58.42" size="1.778" layer="95" xref="yes"/>
 </segment>
 </net>
@@
 <label x="33.02" y="55.88" size="1.778" layer="95" rot="R180" xref="yes"/>
 </segment>
+<segment>
+<pinref part="ENCODER" gate="A" pin="1"/>
+<wire x1="7.62" y1="55.88" x2="12.7" y2="55.88" width="0.1524" layer="91"/>
+<label x="12.7" y="55.88" size="1.778" layer="95" xref="yes"/>
+</segment>
 </net>
 <net name="PB_4" class="0">
@@
 <label x="33.02" y="50.8" size="1.778" layer="95" rot="R180" xref="yes"/>
 </segment>
+<segment>
+<pinref part="ENCODER" gate="A" pin="2"/>
+<wire x1="7.62" y1="58.42" x2="12.7" y2="58.42" width="0.1524" layer="91"/>
+<label x="12.7" y="58.42" size="1.778" layer="95" xref="yes"/>
+</segment>
 </net>
